Commit message: decrease limits by a degree

File: motoman_sda10f_support/urdf/arm_macro.xacro (robot description, xacro)
@@ -111,5 +111,5 @@
       <origin xyz="0.100 ${reflect*0.265} 0.0" rpy="${radians(90)} 0.0 ${(reflect-1)*radians(90)}"/>
       <axis xyz="0 0 ${-reflect}" />
-      <limit lower="${radians(-180)}" upper="${radians(180)}" effort="0" velocity="${radians(170)}" />
+      <limit lower="${radians(-179)}" upper="${radians(179)}" effort="0" velocity="${radians(169)}" />
     </joint>
     <joint name="${prefix}joint_2_l" type="revolute">
@@ -118,5 +118,5 @@
       <origin xyz="0.0 0.0 0.0" rpy="${radians(-90)} 0.0 0.0"/>
       <axis xyz="0 0 ${-reflect}" />
-      <limit lower="${radians(-110)}" upper="${radians(110)}" effort="0" velocity="${radians(170)}" />
+      <limit lower="${radians(-109)}" upper="${radians(109)}" effort="0" velocity="${radians(169)}" />
     </joint>
     <joint name="${prefix}joint_3_e" type="revolute">
@@ -125,5 +125,5 @@
       <origin xyz="0.0 0.360 0.0" rpy="${radians(90)} 0.0 0.0"/>
       <axis xyz="0 0 ${-reflect}" />
-      <limit lower="${radians(-170)}" upper="${radians(170)}" effort="0" velocity="${radians(170)}" />
+      <limit lower="${radians(-169)}" upper="${radians(169)}" effort="0" velocity="${radians(169)}" />
     </joint>
     <joint name="${prefix}joint_4_u" type="revolute">
@@ -132,5 +132,5 @@
       <origin xyz="0.0 0.0 0.0" rpy="${radians(-90)} 0.0 0.0"/>
       <axis xyz="0 0 ${reflect}" />
-      <limit lower="${radians(-135)}" upper="${radians(135)}" effort="0" velocity="${radians(170)}" />
+      <limit lower="${radians(-134)}" upper="${radians(134)}" effort="0" velocity="${radians(169)}" />
     </joint>
     <joint name="${prefix}joint_5_r" type="revolute">
@@ -139,5 +139,5 @@
       <origin xyz="0.0 0.360 0.0" rpy="${radians(90)} 0.0 0.0"/>
       <axis xyz="0 0 ${reflect}" />
-      <limit lower="${radians(-180)}" upper="${radians(180)}" effort="0" velocity="${radians(200)}" />
+      <limit lower="${radians(-179)}" upper="${radians(179)}" effort="0" velocity="${radians(199)}" />
     </joint>
     <joint name="${prefix}joint_6_b" type="revolute">
@@ -146,5 +146,5 @@
       <origin xyz="0.0 0.0 0.0" rpy="${radians(-90)} 0.0 0.0"/>
       <axis xyz="0 0 ${reflect}" />
-      <limit lower="${radians(-110)}" upper="${radians(110)}" effort="0" velocity="${radians(200)}" />
+      <limit lower="${radians(-109)}" upper="${radians(109)}" effort="0" velocity="${radians(199)}" />
     </joint>
     <joint name="${prefix}joint_7_t" type="revolute">
@@ -153,5 +153,5 @@
       <origin xyz="0.0 0.155 0.0" rpy="${radians(-90)} 0.0 0.0"/>
       <axis xyz="0 0 ${-reflect}" />
-      <limit lower="${radians(-180)}" upper="${radians(180)}" effort="0" velocity="${radians(400)}" />
+      <limit lower="${radians(-179)}" upper="${radians(179)}" effort="0" velocity="${radians(399)}" />
     </joint>
     <joint name="${prefix}joint_tool0" type="fixed" >

File: motoman_sda10f_support/urdf/common_torso_macro.xacro (robot description, xacro)
@@ -38,5 +38,5 @@
       <origin xyz="0 0 0" rpy="0 0 0"/>
       <axis xyz="0 0 1" />
-      <limit lower="${radians(-170)}" upper="${radians(170)}" effort="100" velocity="${radians(130)}" />
+      <limit lower="${radians(-90)}" upper="${radians(90)}" effort="100" velocity="${radians(130)}" />
     </joint>
     <joint name="${prefix}joint_b2" type="revolute">
@@ -45,5 +45,5 @@
       <origin xyz="0 0 0" rpy="0 0 0"/>
       <axis xyz="0 0 1" />
-      <limit lower="${radians(-170)}" upper="${radians(170)}" effort="100" velocity="${radians(130)}" />
+      <limit lower="${radians(-90)}" upper="${radians(90)}" effort="100" velocity="${radians(130)}" />
       <mimic joint="${prefix}joint_b1" multiplier="1" offset="0"/>
     </joint>

Commit message: lower joint limits and reduce camera size

File: motoman_sda10f_support/urdf/arm_macro.xacro (robot description, xacro)
@@ -111,5 +111,5 @@
       <origin xyz="0.100 ${reflect*0.265} 0.0" rpy="${radians(90)} 0.0 ${(reflect-1)*radians(90)}"/>
       <axis xyz="0 0 ${-reflect}" />
-      <limit lower="${radians(-179)}" upper="${radians(179)}" effort="0" velocity="${radians(169)}" />
+      <limit lower="${radians(-178)}" upper="${radians(178)}" effort="0" velocity="${radians(169)}" />
     </joint>
     <joint name="${prefix}joint_2_l" type="revolute">
@@ -118,5 +118,5 @@
       <origin xyz="0.0 0.0 0.0" rpy="${radians(-90)} 0.0 0.0"/>
       <axis xyz="0 0 ${-reflect}" />
-      <limit lower="${radians(-109)}" upper="${radians(109)}" effort="0" velocity="${radians(169)}" />
+      <limit lower="${radians(-108)}" upper="${radians(108)}" effort="0" velocity="${radians(169)}" />
     </joint>
     <joint name="${prefix}joint_3_e" type="revolute">
@@ -125,5 +125,5 @@
       <origin xyz="0.0 0.360 0.0" rpy="${radians(90)} 0.0 0.0"/>
       <axis xyz="0 0 ${-reflect}" />
-      <limit lower="${radians(-169)}" upper="${radians(169)}" effort="0" velocity="${radians(169)}" />
+      <limit lower="${radians(-168)}" upper="${radians(168)}" effort="0" velocity="${radians(169)}" />
     </joint>
     <joint name="${prefix}joint_4_u" type="revolute">
@@ -132,5 +132,5 @@
       <origin xyz="0.0 0.0 0.0" rpy="${radians(-90)} 0.0 0.0"/>
       <axis xyz="0 0 ${reflect}" />
-      <limit lower="${radians(-134)}" upper="${radians(134)}" effort="0" velocity="${radians(169)}" />
+      <limit lower="${radians(-133)}" upper="${radians(133)}" effort="0" velocity="${radians(169)}" />
     </joint>
     <joint name="${prefix}joint_5_r" type="revolute">
@@ -139,5 +139,5 @@
       <origin xyz="0.0 0.360 0.0" rpy="${radians(90)} 0.0 0.0"/>
       <axis xyz="0 0 ${reflect}" />
-      <limit lower="${radians(-179)}" upper="${radians(179)}" effort="0" velocity="${radians(199)}" />
+      <limit lower="${radians(-178)}" upper="${radians(178)}" effort="0" velocity="${radians(199)}" />
     </joint>
     <joint name="${prefix}joint_6_b" type="revolute">
@@ -146,5 +146,5 @@
       <origin xyz="0.0 0.0 0.0" rpy="${radians(-90)} 0.0 0.0"/>
       <axis xyz="0 0 ${reflect}" />
-      <limit lower="${radians(-109)}" upper="${radians(109)}" effort="0" velocity="${radians(199)}" />
+      <limit lower="${radians(-108)}" upper="${radians(108)}" effort="0" velocity="${radians(199)}" />
     </joint>
     <joint name="${prefix}joint_7_t" type="revolute">
@@ -153,5 +153,5 @@
       <origin xyz="0.0 0.155 0.0" rpy="${radians(-90)} 0.0 0.0"/>
       <axis xyz="0 0 ${-reflect}" />
-      <limit lower="${radians(-179)}" upper="${radians(179)}" effort="0" velocity="${radians(399)}" />
+      <limit lower="${radians(-178)}" upper="${radians(178)}" effort="0" velocity="${radians(399)}" />
     </joint>
     <joint name="${prefix}joint_tool0" type="fixed" >

File: motoman_sda10f_support/urdf/sda10f.xacro (robot description, xacro)
@@ -70,5 +70,5 @@
 			<origin rpy="0 0 0" xyz="0 0 0" />
 			<geometry>
-				<box size="0.1 0.15 0.1" />
+				<box size="0.1 0.15 0.05" />
 			</geometry>
 			<material name="">
@@ -79,5 +79,5 @@
 			<origin rpy="0 0 0" xyz="0 0 0" />
 			<geometry>
-				<box size="0.1 0.15 0.1" />
+				<box size="0.1 0.15 0.05" />
 			</geometry>
 		</collision>
@@ -86,5 +86,5 @@
 		<parent link="arm_right_link_6_b" />
 		<child link="camera_arm_link" />
-		<origin rpy="0 0 0" xyz="0 0.03 0.125" />
+		<origin rpy="0 0 0" xyz="0 0.02 0.1" />
 	</joint>
 </robot>

Commit message: update camera mount

File: motoman_sda10f_support/urdf/arm_macro.xacro (robot description, xacro)
@@ -111,5 +111,5 @@
       <origin xyz="0.100 ${reflect*0.265} 0.0" rpy="${radians(90)} 0.0 ${(reflect-1)*radians(90)}"/>
       <axis xyz="0 0 ${-reflect}" />
-      <limit lower="${radians(-178)}" upper="${radians(178)}" effort="0" velocity="${radians(169)}" />
+      <limit lower="${radians(-177)}" upper="${radians(177)}" effort="0" velocity="${radians(169)}" />
     </joint>
     <joint name="${prefix}joint_2_l" type="revolute">
@@ -139,5 +139,5 @@
       <origin xyz="0.0 0.360 0.0" rpy="${radians(90)} 0.0 0.0"/>
       <axis xyz="0 0 ${reflect}" />
-      <limit lower="${radians(-178)}" upper="${radians(178)}" effort="0" velocity="${radians(199)}" />
+      <limit lower="${radians(-177)}" upper="${radians(177)}" effort="0" velocity="${radians(199)}" />
     </joint>
     <joint name="${prefix}joint_6_b" type="revolute">
@@ -153,5 +153,5 @@
       <origin xyz="0.0 0.155 0.0" rpy="${radians(-90)} 0.0 0.0"/>
       <axis xyz="0 0 ${-reflect}" />
-      <limit lower="${radians(-178)}" upper="${radians(178)}" effort="0" velocity="${radians(399)}" />
+      <limit lower="${radians(-177)}" upper="${radians(177)}" effort="0" velocity="${radians(399)}" />
     </joint>
     <joint name="${prefix}joint_tool0" type="fixed" >

File: motoman_sda10f_support/urdf/sda10f.xacro (robot description, xacro)
@@ -70,5 +70,5 @@
 			<origin rpy="0 0 0" xyz="0 0 0" />
 			<geometry>
-				<box size="0.1 0.15 0.05" />
+				<box size="0.12 0.15 0.05" />
 			</geometry>
 			<material name="">
@@ -86,5 +86,5 @@
 		<parent link="arm_right_link_6_b" />
 		<child link="camera_arm_link" />
-		<origin rpy="0 0 0" xyz="0 0.02 0.1" />
+		<origin rpy="0 0 0" xyz="0 0.05 0.1" />
 	</joint>
 </robot>
