Commit message: rotate gripper

File: motoman_sda10f_moveit_config/config/gazebo_motoman_sda10f.urdf (robot description, URDF)
Before this commit: robot motoman_sda10f, 32 links, 31 joints
Links:
- added link motoman_left_ee
Joints:
- added joint motoman_left_joint_ee: type fixed, parent arm_left_link_tool0, child motoman_left_ee, origin xyz=0 0 0 rpy=0 0 0
- joint motoman_right_joint_pre_ee: origin xyz=0 0 0 rpy=0 0 0 -> xyz=0 0 0 rpy=0 0 1.5708

File: motoman_sda10f_support/urdf/sda10f.xacro (robot description, xacro)
@@ -8,5 +8,5 @@
 		<parent link="arm_right_link_tool0"/>
 		<child link="robotiq_arg2f_base_link"/>
-		<origin xyz="0 0 0" rpy="0 0 0" />
+		<origin xyz="0 0 0" rpy="0 0 1.5708" />
 	</joint>
 	<joint name="motoman_right_joint_ee" type="fixed">
@@ -16,3 +16,9 @@
 	</joint>
 	<link name="motoman_right_ee"></link>
+	<joint name="motoman_left_joint_ee" type="fixed">
+		<parent link="arm_left_link_tool0" />
+		<child link="motoman_left_ee" />
+		<origin rpy="0 0 0" xyz="0 0 0" />
+	</joint>
+	<link name="motoman_left_ee" />
 </robot>

Commit message: update gazebo urdf

File: motoman_sda10f_moveit_config/config/gazebo_motoman_sda10f.urdf (robot description, URDF)
Before this commit: robot motoman_sda10f, 33 links, 32 joints
Links:
- added link camera_arm_link, mass 0.1; collision box size=0.1 0.15 0.05; visual box size=0.12 0.15 0.05
- added link camera_torso_link, mass 0.1; collision cylinder length=0.12 radius=0.08; visual cylinder length=0.12 radius=0.08
- added link robotiq_arg2f_extra_link, mass 0.1; collision cylinder length=0.017 radius=0.04; visual cylinder length=0.017 radius=0.04
Joints:
- added joint camera_arm_joint: type fixed, parent arm_right_link_6_b, child camera_arm_link, origin xyz=0 0.05 0.1 rpy=0 0 0
- added joint camera_torso_joint: type fixed, parent torso_link_b1, child camera_torso_link, origin xyz=0.1 0.0 0.2 rpy=0 0 0
- added joint motoman_right_joint_ee_extra: type fixed, parent robotiq_arg2f_extra_link, child robotiq_arg2f_base_link, origin xyz=0 0 0.0085 rpy=0 0 0
- joint arm_left_joint_1_s: limit lower=-3.141592653589793 upper=3.141592653589793 effort=0 velocity=2.9670597283903604 -> lower=-3.0892327760299634 upper=3.0892327760299634 effort=0 velocity=2.949606435870417
- joint arm_left_joint_2_l: limit lower=-1.9198621771937625 upper=1.9198621771937625 effort=0 velocity=2.9670597283903604 -> lower=-1.8849555921538759 upper=1.8849555921538759 effort=0 velocity=2.949606435870417
- joint arm_left_joint_3_e: limit lower=-2.9670597283903604 upper=2.9670597283903604 effort=0 velocity=2.9670597283903604 -> lower=-2.9321531433504737 upper=2.9321531433504737 effort=0 velocity=2.949606435870417
- joint arm_left_joint_4_u: limit lower=-2.356194490192345 upper=2.356194490192345 effort=0 velocity=2.9670597283903604 -> lower=-2.321287905152458 upper=2.321287905152458 effort=0 velocity=2.949606435870417
- joint arm_left_joint_5_r: limit lower=-3.141592653589793 upper=3.141592653589793 effort=0 velocity=3.490658503988659 -> lower=-3.0892327760299634 upper=3.0892327760299634 effort=0 velocity=3.473205211468716
- joint arm_left_joint_6_b: limit lower=-1.9198621771937625 upper=1.9198621771937625 effort=0 velocity=3.490658503988659 -> lower=-1.8849555921538759 upper=1.8849555921538759 effort=0 velocity=3.473205211468716
- joint arm_left_joint_7_t: limit lower=-3.141592653589793 upper=3.141592653589793 effort=0 velocity=6.981317007977318 -> lower=-3.0892327760299634 upper=3.0892327760299634 effort=0 velocity=6.963863715457375
- joint arm_right_joint_1_s: limit lower=-3.141592653589793 upper=3.141592653589793 effort=0 velocity=2.9670597283903604 -> lower=-3.0892327760299634 upper=3.0892327760299634 effort=0 velocity=2.949606435870417
- joint arm_right_joint_2_l: limit lower=-1.9198621771937625 upper=1.9198621771937625 effort=0 velocity=2.9670597283903604 -> lower=-1.8849555921538759 upper=1.8849555921538759 effort=0 velocity=2.949606435870417
- joint arm_right_joint_3_e: limit lower=-2.9670597283903604 upper=2.9670597283903604 effort=0 velocity=2.9670597283903604 -> lower=-2.9321531433504737 upper=2.9321531433504737 effort=0 velocity=2.949606435870417
- joint arm_right_joint_4_u: limit lower=-2.356194490192345 upper=2.356194490192345 effort=0 velocity=2.9670597283903604 -> lower=-2.321287905152458 upper=2.321287905152458 effort=0 velocity=2.949606435870417
- joint arm_right_joint_5_r: limit lower=-3.141592653589793 upper=3.141592653589793 effort=0 velocity=3.490658503988659 -> lower=-3.0892327760299634 upper=3.0892327760299634 effort=0 velocity=3.473205211468716
- joint arm_right_joint_6_b: limit lower=-1.9198621771937625 upper=1.9198621771937625 effort=0 velocity=3.490658503988659 -> lower=-1.8849555921538759 upper=1.8849555921538759 effort=0 velocity=3.473205211468716
- joint arm_right_joint_7_t: limit lower=-3.141592653589793 upper=3.141592653589793 effort=0 velocity=6.981317007977318 -> lower=-3.0892327760299634 upper=3.0892327760299634 effort=0 velocity=6.963863715457375
- joint motoman_right_joint_pre_ee: child robotiq_arg2f_base_link -> robotiq_arg2f_extra_link; origin xyz=0 0 0 rpy=0 0 1.5708 -> xyz=0 0 0.0085 rpy=0 0 1.5708
- joint torso_joint_b1: limit lower=-2.9670597283903604 upper=2.9670597283903604 effort=100 velocity=2.2689280275926285 -> lower=-1.5707963267948966 upper=1.5707963267948966 effort=100 velocity=2.2689280275926285
- joint torso_joint_b2: limit lower=-2.9670597283903604 upper=2.9670597283903604 effort=100 velocity=2.2689280275926285 -> lower=-1.5707963267948966 upper=1.5707963267948966 effort=100 velocity=2.2689280275926285

Commit message: comment out camera_arm_link

File: motoman_sda10f_moveit_config/config/gazebo_motoman_sda10f.urdf (robot description, URDF)
Before this commit: robot motoman_sda10f, 36 links, 35 joints
Links:
- removed link camera_arm_link
Joints:
- removed joint camera_arm_joint

File: motoman_sda10f_support/urdf/sda10f.xacro (robot description, xacro)
@@ -25,5 +25,5 @@
 		<parent link="arm_right_link_tool0"/>
 		<child link="robotiq_arg2f_extra_link"/>
-    <origin xyz="0 0 0.0085" rpy="0 0 1.5708" />
+		<origin xyz="0 0 0.0085" rpy="0 0 1.5708" />
 	</joint>
 	<joint name="motoman_right_joint_ee_extra" type="fixed">
@@ -66,4 +66,5 @@
 		<origin rpy="0 0 0" xyz="0.1 0.0 0.2" />
 	</joint>
+	<!--
 	<link name="camera_arm_link" >
 		<visual>
@@ -88,3 +89,4 @@
 		<origin rpy="0 0 0" xyz="0 -0.055 0.04" />
 	</joint>
+	-->
 </robot>
